File: birdEar/MCU.sch (KiCad schematic (older format))
At the start: 15 parts

Commit message: Worked on the HW and made some changes to the IOC file.
Parts:
- added C18, C20: 1uF, symbol Device:C_Small
- added C19: 2.2uF, symbol Device:C_Small
- added C21: 4.7uF, symbol Device:C_Small
- added C22: 100uF, symbol Device:C_Small
- added D1, D2, D3: LED, symbol Device:LED
- added J1: Conn_01x03, symbol Connector_Generic:Conn_01x03
- added J3: SWD, symbol Connector_Generic:Conn_02x03_Counter_Clockwise
- added R10, R11, R12, R5, R6, R7, R8, R9: 47K, symbol Device:R_Small_US
- added SW1, SW2, SW3: SW_Push_Dual, symbol Switch:SW_Push_Dual
- J2: renamed from J?; symbol Connector:Micro_SD_Card_Det_Hirose_DM3AT -> birdEar-rescue:Micro_SD_Card_Det_Hirose_DM3AT-Connector
- gave numbers to parts that had none: 14
Connections:
- net labels added: Audio_In, CLK, CMD, DAT0, DAT1, DAT2, DAT3, Loud, PB1, PB2, SD_DET, SWCLK, SWDIO, SW_RST, UART_RX, UART_TX
- wire segments 107 -> 241

Commit message: Added some parts to the schematic, maps some parts to their footprints. You know.
Parts:
- removed SW2, SW3: SW_Push_Dual, symbol Switch:SW_Push_Dual
- added SW4: SW_Push, symbol Switch:SW_Push
- C10, C11, C12, C13, C14, C15, C16, C17, C18, C19, C20, C21, C22, C5, C6, C7, C8, C9: footprint (none) -> Capacitor_SMD:C_0805_2012Metric
- D1, D2, D3: footprint (none) -> LED_SMD:LED_0805_2012Metric
- J1: footprint (none) -> Connector_PinHeader_2.54mm:PinHeader_1x03_P2.54mm_Vertical
- J2: footprint (none) -> Connector_Card:microSD_HC_Hirose_DM3AT-SF-PEJM5
- J3: footprint (none) -> Connector_PinHeader_2.54mm:PinHeader_2x03_P2.54mm_Vertical
- R10, R11, R12: value 47K -> 1K; footprint (none) -> Resistor_SMD:R_0805_2012Metric
- R5, R6, R7, R8, R9: footprint (none) -> Resistor_SMD:R_0805_2012Metric
Connections:
- net I2C_SCL: now reaches U3.136 (PB6)
- net I2C_SDA: now reaches U3.137 (PB7)

Commit message: Hardware is almost finished
Parts:
- removed SW1: SW_Push_Dual, symbol Switch:SW_Push_Dual
- added J5: Conn_01x08_Male, Connector_PinHeader_2.54mm:PinHeader_1x08_P2.54mm_Vertical, symbol Connector:Conn_01x08_Male
- J2: symbol birdEar-rescue:Micro_SD_Card_Det_Hirose_DM3AT-Connector -> birdEar-rescue:Micro_SD_Card_Det_Hirose_DM3AT-Connector-birdEar-rescue
- SW4: value SW_Push -> KSA0A311 LFTR; footprint (none) -> Button_Switch_THT:SW_Tactile_Straight_KSA0Axx1LFTR
Connections:
- net GND: now also SW4.1, J5.8 (Pin_8)
- net PB1: now also U3.1 (PE2); no longer U3.142 (PE1)
- net PB2: now also U3.2 (PE3); no longer U3.1 (PE2)
- net at U3.25 (NRST): now also SW4.2
- net PF13: now reaches U3.53 (PF13)
- net PF13: now also J5.1 (Pin_1)
- net PF14: now reaches U3.54 (PF14)
- net PF14: now also J5.2 (Pin_2)
- net PF15: now reaches U3.55 (PF15)
- net PF15: now also J5.3 (Pin_3)
- net PG0: now reaches U3.56 (PG0)
- net PG0: now also J5.4 (Pin_4)
- net PG1: now reaches U3.57 (PG1)
- net PG1: now also J5.5 (Pin_5)
- net PE7: now reaches U3.58 (PE7)
- net PE7: now also J5.6 (Pin_6)
- net PE8: now reaches U3.59 (PE8)
- net PE8: now also J5.7 (Pin_7)
- net PE9: now reaches U3.60 (PE9)
Other:
- moved on the sheet: SW4
Changed lines of the file:
@@
 EESchema Schematic File Version 4
 LIBS:birdEar-cache
-EELAYER 30 0
+EELAYER 26 0
 EELAYER END
 $Descr A4 11693 8268
@@
 $EndComp
 $Comp
-L birdEar-rescue:Micro_SD_Card_Det_Hirose_DM3AT-Connector J?
+L birdEar-rescue:Micro_SD_Card_Det_Hirose_DM3AT-Connector-birdEar-rescue J?
 U 1 1 5D8C50AB
 P 2250 6550
@@
 	2800 2450 2800 2200
 $Comp
-L Switch:SW_Push_Dual SW1
-U 1 1 5DAF0B9D
-P 2200 2100
-F 0 "SW1" H 2200 2385 50  0000 C CNN
-F 1 "SW_Push_Dual" H 2200 2294 50  0000 C CNN
-F 2 "" H 2200 2300 50  0001 C CNN
-F 3 "~" H 2200 2300 50  0001 C CNN
-	1    2200 2100
-	1    0    0    -1
-$EndComp
-Wire Wire Line
-	2400 2100 2500 2100
-Wire Wire Line
-	2500 2100 2500 2200
-Wire Wire Line
-	2500 2300 2400 2300
-Wire Wire Line
-	2500 2200 2800 2200
-Connection ~ 2500 2200
-Wire Wire Line
-	2500 2200 2500 2300
-Wire Wire Line
-	2000 2100 1900 2100
-Wire Wire Line
-	1900 2100 1900 2200
-Wire Wire Line
-	1900 2300 2000 2300
-$Comp
 L power:GND #PWR018
 U 1 1 5DB0AF39
@@
 Wire Wire Line
 	1750 2350 1750 2200
-Wire Wire Line
-	1750 2200 1900 2200
-Connection ~ 1900 2200
-Wire Wire Line
-	1900 2200 1900 2300
 $Comp
 L power:+3.3V #PWR021
@@
 	3650 2300 3650 2200
 Wire Wire Line
-	8000 2150 8000 2450
+	8100 2150 8100 2450
 $Comp
 L Device:LED D1
@@
 Text HLabel 5200 5300 3    50   Input ~ 0
 I2C_SDA
-Text HLabel 8000 2150 1    50   Input ~ 0
+Text HLabel 8100 2150 1    50   Input ~ 0
 PB1
-Text HLabel 8100 2150 1    50   Input ~ 0
+Text HLabel 8200 2150 1    50   Input ~ 0
 PB2
 Wire Wire Line
-	8100 2150 8100 2450
+	8200 2150 8200 2450
 $Comp
 L Switch:SW_Push SW4
 U 1 1 5DA7B1B6
-P 2200 1250
-F 0 "SW4" H 2200 1535 50  0000 C CNN
-F 1 "SW_Push" H 2200 1444 50  0000 C CNN
-F 2 "" H 2200 1450 50  0001 C CNN
-F 3 "~" H 2200 1450 50  0001 C CNN
-	1    2200 1250
-	1    0    0    -1
-$EndComp
+P 2200 2200
+F 0 "SW4" H 2200 2485 50  0000 C CNN
+F 1 "KSA0A311 LFTR" H 2200 2394 50  0000 C CNN
+F 2 "Button_Switch_THT:SW_Tactile_Straight_KSA0Axx1LFTR" H 2200 2400 50  0001 C CNN
+F 3 "~" H 2200 2400 50  0001 C CNN
+	1    2200 2200
+	1    0    0    -1
+$EndComp
+Wire Wire Line
+	2400 2200 2800 2200
+Wire Wire Line
+	1750 2200 2000 2200
+Wire Wire Line
+	7500 2450 7500 2150
+Wire Wire Line
+	7600 2450 7600 2150
+Text Label 7500 2150 1    50   ~ 0
+PF13
+Text Label 7600 2150 1    50   ~ 0
+PF14
+Wire Wire Line
+	10100 1450 9800 1450
+Wire Wire Line
+	10100 1550 9800 1550
+Text Label 9800 1450 2    50   ~ 0
+PF13
+Text Label 9800 1550 2    50   ~ 0
+PF14
+Wire Wire Line
+	7700 2450 7700 2150
+Text Label 7700 2150 1    50   ~ 0
+PF15
+Wire Wire Line
+	4500 2450 4500 2150
+Text Label 4500 2150 1    50   ~ 0
+PG0
+Wire Wire Line
+	10100 1650 9800 1650
+Text Label 9800 1650 2    50   ~ 0
+PF15
+Wire Wire Line
+	10100 1750 9800 1750
+Text Label 9800 1750 2    50   ~ 0
+PG0
+Wire Wire Line
+	4600 2450 4600 2150
+Text Label 4600 2150 1    50   ~ 0
+PG1
+Wire Wire Line
+	8600 2450 8600 2150
+Text Label 8600 2150 1    50   ~ 0
+PE7
+Wire Wire Line
+	10100 1850 9800 1850
+Text Label 9800 1850 2    50   ~ 0
+PG1
+Wire Wire Line
+	10100 1950 9800 1950
+Text Label 9800 1950 2    50   ~ 0
+PE7
+Wire Wire Line
+	8700 2450 8700 2150
+Text Label 8700 2150 1    50   ~ 0
+PE8
+Wire Wire Line
+	8800 2450 8800 2150
+Text Label 8800 2150 1    50   ~ 0
+PE9
+Wire Wire Line
+	10100 2050 9800 2050
+Text Label 9800 2050 2    50   ~ 0
+PE8
+$Comp
+L Connector:Conn_01x08_Male J5
+U 1 1 5DB1E831
+P 10300 1750
+F 0 "J5" H 10273 1723 50  0000 R CNN
+F 1 "Conn_01x08_Male" H 10273 1632 50  0000 R CNN
+F 2 "Connector_PinHeader_2.54mm:PinHeader_1x08_P2.54mm_Vertical" H 10300 1750 50  0001 C CNN
+F 3 "~" H 10300 1750 50  0001 C CNN
+	1    10300 1750
+	-1   0    0    -1
+$EndComp
+Wire Wire Line
+	10100 2150 9800 2150
+Wire Wire Line
+	9800 2150 9800 2250
+$Comp
+L power:GND #PWR0104
+U 1 1 5DB6A181
+P 9800 2250
+F 0 "#PWR0104" H 9800 2000 50  0001 C CNN
+F 1 "GND" H 9805 2077 50  0000 C CNN
+F 2 "" H 9800 2250 50  0001 C CNN
+F 3 "" H 9800 2250 50  0001 C CNN
+	1    9800 2250
+	1    0    0    -1
+$EndComp

Commit message: Implemented anti aliasing filter, worked on the layout, added some gnd points
Parts:
- removed J3: SWD, Connector_PinHeader_2.54mm:PinHeader_2x03_P2.54mm_Vertical, symbol Connector_Generic:Conn_02x03_Counter_Clockwise
- added J3: Conn_02x03_Odd_Even, Connector_PinHeader_2.54mm:PinHeader_2x03_P2.54mm_Vertical, symbol Connector_Generic:Conn_02x03_Odd_Even
- J2: symbol birdEar-rescue:Micro_SD_Card_Det_Hirose_DM3AT-Connector-birdEar-rescue -> birdEar-rescue:Micro_SD_Card_Det_Hirose_DM3AT-Connector-birdEar-rescue-birdEar-rescue
Connections:
- net +3V3: now also J3.1 (Pin_1)
- net GND: now also J3.5 (Pin_5)
- net SWCLK: now also J3.4 (Pin_4)
- net SWDIO: now also J3.2 (Pin_2)
- net SW_RST: now also J3.3 (Pin_3)
Changed lines of the file:
@@
 EESchema Schematic File Version 4
 LIBS:birdEar-cache
-EELAYER 26 0
+EELAYER 30 0
 EELAYER END
 $Descr A4 11693 8268
@@
 $EndComp
 $Comp
-L birdEar-rescue:Micro_SD_Card_Det_Hirose_DM3AT-Connector-birdEar-rescue J?
+L birdEar-rescue:Micro_SD_Card_Det_Hirose_DM3AT-Connector-birdEar-rescue-birdEar-rescue J?
 U 1 1 5D8C50AB
 P 2250 6550
@@
 Text Label 4900 1250 2    50   ~ 0
 SW_RST
-$Comp
-L Connector_Generic:Conn_02x03_Counter_Clockwise J3
-U 1 1 5DA958CC
-P 5200 1250
-F 0 "J3" H 5250 1450 50  0000 C CNN
-F 1 "SWD" H 5250 1050 50  0000 C CNN
-F 2 "Connector_PinHeader_2.54mm:PinHeader_2x03_P2.54mm_Vertical" H 5200 1250 50  0001 C CNN
-F 3 "~" H 5200 1250 50  0001 C CNN
-	1    5200 1250
-	1    0    0    -1
-$EndComp
 Wire Wire Line
 	5600 1150 5500 1150
@@
 	1    0    0    -1
 $EndComp
+$Comp
+L Connector_Generic:Conn_02x03_Odd_Even J3
+U 1 1 5DA504A4
+P 5200 1250
+F 0 "J3" H 5250 1567 50  0000 C CNN
+F 1 "Conn_02x03_Odd_Even" H 5250 1476 50  0000 C CNN
+F 2 "Connector_PinHeader_2.54mm:PinHeader_2x03_P2.54mm_Vertical" H 5200 1250 50  0001 C CNN
+F 3 "~" H 5200 1250 50  0001 C CNN
+	1    5200 1250
+	1    0    0    -1
+$EndComp
