File: birdEar/birdEar.sch (KiCad schematic (older format))
At the start: 18 parts

Commit message: Worked on the HW and made some changes to the IOC file.
Parts:
- gave numbers to parts that had none: 14
Other:
- note added: "STM32"
Changed lines of the file:
@@
 EESchema Schematic File Version 4
-EELAYER 26 0
+LIBS:birdEar-cache
+EELAYER 30 0
 EELAYER END
 $Descr USLetter 11000 8500
@@
 $EndDescr
 $Comp
-L Device:Microphone MK?
+L Device:Microphone MK1
 U 1 1 5D8C2F06
 P 850 3700
-F 0 "MK?" H 980 3746 50  0000 L CNN
+F 0 "MK1" H 980 3746 50  0000 L CNN
 F 1 "CMA-4544PF-W" H 980 3655 50  0000 L CNN
 F 2 "" V 850 3800 50  0001 C CNN
@@
 $EndComp
 $Comp
-L Device:Battery_Cell BT?
+L Device:Battery_Cell BT1
 U 1 1 5D8C35FD
 P 1200 1600
-F 0 "BT?" H 1318 1696 50  0000 L CNN
+F 0 "BT1" H 1318 1696 50  0000 L CNN
 F 1 "Battery_Cell" H 1318 1605 50  0000 L CNN
 F 2 "" V 1200 1660 50  0001 C CNN
@@
 F0 "MCU" 50
 F1 "MCU.sch" 50
+F2 "Audio_In" I L 6450 3600 50
+F3 "Loud" I L 6450 3700 50
 $EndSheet
 $Comp
-L Regulator_Linear:AZ1117-3.3 U?
+L Regulator_Linear:AZ1117-3.3 U2
 U 1 1 5D8C3D0D
 P 2650 1350
-F 0 "U?" H 2650 1592 50  0000 C CNN
+F 0 "U2" H 2650 1592 50  0000 C CNN
 F 1 "AZ1117EH-3.3TRG1" H 2650 1501 50  0000 C CNN
 F 2 "" H 2650 1600 50  0001 C CIN
@@
 $EndComp
 $Comp
-L power:GND #PWR?
+L power:GND #PWR011
 U 1 1 5D8C40B1
 P 2650 1800
-F 0 "#PWR?" H 2650 1550 50  0001 C CNN
+F 0 "#PWR011" H 2650 1550 50  0001 C CNN
 F 1 "GND" H 2655 1627 50  0000 C CNN
 F 2 "" H 2650 1800 50  0001 C CNN
@@
 $EndComp
 $Comp
-L Device:C_Small C?
+L Device:C_Small C3
 U 1 1 5D8C4221
 P 2050 1550
-F 0 "C?" H 2150 1600 50  0000 L CNN
+F 0 "C3" H 2150 1600 50  0000 L CNN
 F 1 "1uF" H 2142 1505 50  0000 L CNN
 F 2 "" H 2050 1550 50  0001 C CNN
@@
 	2050 1750 2050 1650
 $Comp
-L Device:C_Small C?
+L Device:C_Small C4
 U 1 1 5D8C447C
 P 3250 1550
-F 0 "C?" H 3350 1600 50  0000 L CNN
+F 0 "C4" H 3350 1600 50  0000 L CNN
 F 1 "1uF" H 3342 1505 50  0000 L CNN
 F 2 "" H 3250 1550 50  0001 C CNN
@@
 Connection ~ 2050 1750
 $Comp
-L power:+3.3V #PWR?
+L power:+3.3V #PWR012
 U 1 1 5D8C4A64
 P 3250 1250
-F 0 "#PWR?" H 3250 1100 50  0001 C CNN
+F 0 "#PWR012" H 3250 1100 50  0001 C CNN
 F 1 "+3.3V" H 3265 1423 50  0000 C CNN
 F 2 "" H 3250 1250 50  0001 C CNN
@@
 	850  3900 850  4050
 $Comp
-L power:GND #PWR?
+L power:GND #PWR01
 U 1 1 5D8C4D2E
 P 850 4050
-F 0 "#PWR?" H 850 3800 50  0001 C CNN
+F 0 "#PWR01" H 850 3800 50  0001 C CNN
 F 1 "GND" H 855 3877 50  0000 C CNN
 F 2 "" H 850 4050 50  0001 C CNN
@@
 	850  3500 850  3300
 $Comp
-L Amplifier_Operational:LM324 U?
+L Amplifier_Operational:LM324 U1
 U 1 1 5D8C521D
 P 2850 3200
-F 0 "U?" H 2850 2833 50  0000 C CNN
+F 0 "U1" H 2850 2833 50  0000 C CNN
 F 1 "LM324" H 2850 2924 50  0000 C CNN
 F 2 "" H 2800 3300 50  0001 C CNN
@@
 $EndComp
 $Comp
-L Amplifier_Operational:LM324 U?
+L Amplifier_Operational:LM324 U1
 U 2 1 5D8C52C4
 P 2950 4950
-F 0 "U?" H 2950 5317 50  0000 C CNN
+F 0 "U1" H 2950 5317 50  0000 C CNN
 F 1 "LM324" H 2950 5226 50  0000 C CNN
 F 2 "" H 2900 5050 50  0001 C CNN
@@
 $EndComp
 $Comp
-L Amplifier_Operational:LM324 U?
+L Amplifier_Operational:LM324 U1
 U 3 1 5D8C5364
 P 2950 6250
-F 0 "U?" H 2950 6617 50  0000 C CNN
+F 0 "U1" H 2950 6617 50  0000 C CNN
 F 1 "LM324" H 2950 6526 50  0000 C CNN
 F 2 "" H 2900 6350 50  0001 C CNN
@@
 $EndComp
 $Comp
-L Amplifier_Operational:LM324 U?
+L Amplifier_Operational:LM324 U1
 U 4 1 5D8C5409
 P 2900 7050
-F 0 "U?" H 2900 7417 50  0000 C CNN
+F 0 "U1" H 2900 7417 50  0000 C CNN
 F 1 "LM324" H 2900 7326 50  0000 C CNN
 F 2 "" H 2850 7150 50  0001 C CNN
@@
 $EndComp
 $Comp
-L Amplifier_Operational:LM324 U?
+L Amplifier_Operational:LM324 U1
 U 5 1 5D8C54A9
 P 950 5400
-F 0 "U?" H 550 5450 50  0000 L CNN
+F 0 "U1" H 550 5450 50  0000 L CNN
 F 1 "LM324" H 550 5350 50  0000 L CNN
 F 2 "" H 900 5500 50  0001 C CNN
@@
 	850  5700 850  5850
 $Comp
-L power:GND #PWR?
+L power:GND #PWR03
 U 1 1 5D8C59B1
 P 850 5850
-F 0 "#PWR?" H 850 5600 50  0001 C CNN
+F 0 "#PWR03" H 850 5600 50  0001 C CNN
 F 1 "GND" H 855 5677 50  0000 C CNN
 F 2 "" H 850 5850 50  0001 C CNN
@@
 $EndComp
 $Comp
-L power:+3.3V #PWR?
+L power:+3.3V #PWR02
 U 1 1 5D8C5AA2
 P 850 4950
-F 0 "#PWR?" H 850 4800 50  0001 C CNN
+F 0 "#PWR02" H 850 4800 50  0001 C CNN
 F 1 "+3.3V" H 865 5123 50  0000 C CNN
 F 2 "" H 850 4950 50  0001 C CNN
@@
 $EndComp
 $Comp
-L Device:R_Small_US R?
+L Device:R_Small_US R1
 U 1 1 5D8C65A2
 P 1100 3100
-F 0 "R?" H 1168 3146 50  0000 L CNN
+F 0 "R1" H 1168 3146 50  0000 L CNN
 F 1 "2.2k" H 1168 3055 50  0000 L CNN
 F 2 "" H 1100 3100 50  0001 C CNN
@@
 $EndComp
 $Comp
-L Device:C_Small C?
+L Device:C_Small C2
 U 1 1 5D8C666E
 P 1300 3300
-F 0 "C?" H 1400 3350 50  0000 L CNN
+F 0 "C2" H 1400 3350 50  0000 L CNN
 F 1 "1uF" H 1392 3255 50  0000 L CNN
 F 2 "" H 1300 3300 50  0001 C CNN
@@
 $EndComp
 $Comp
-L power:+3.3V #PWR?
+L power:+3.3V #PWR04
 U 1 1 5D8C70F2
 P 1100 2900
-F 0 "#PWR?" H 1100 2750 50  0001 C CNN
+F 0 "#PWR04" H 1100 2750 50  0001 C CNN
 F 1 "+3.3V" H 1115 3073 50  0000 C CNN
 F 2 "" H 1100 2900 50  0001 C CNN
@@
 	1100 3300 1200 3300
 $Comp
-L Device:R_Small_US R?
+L Device:R_Small_US R2
 U 1 1 5D8C8826
 P 1850 3050
-F 0 "R?" H 1918 3096 50  0000 L CNN
+F 0 "R2" H 1918 3096 50  0000 L CNN
 F 1 "1M" H 1918 3005 50  0000 L CNN
 F 2 "" H 1850 3050 50  0001 C CNN
@@
 $EndComp
 $Comp
-L Device:R_Small_US R?
+L Device:R_Small_US R3
 U 1 1 5D8C88C0
 P 1850 3550
-F 0 "R?" H 1918 3596 50  0000 L CNN
+F 0 "R3" H 1918 3596 50  0000 L CNN
 F 1 "1M" H 1918 3505 50  0000 L CNN
 F 2 "" H 1850 3550 50  0001 C CNN
@@
 Connection ~ 1850 3300
 $Comp
-L power:GND #PWR?
+L power:GND #PWR07
 U 1 1 5D8C93C4
 P 1850 3750
-F 0 "#PWR?" H 1850 3500 50  0001 C CNN
+F 0 "#PWR07" H 1850 3500 50  0001 C CNN
 F 1 "GND" H 1855 3577 50  0000 C CNN
 F 2 "" H 1850 3750 50  0001 C CNN
@@
 	1850 2850 1850 2950
 $Comp
-L power:+3.3V #PWR?
+L power:+3.3V #PWR06
 U 1 1 5D8C9BE2
 P 1850 2850
-F 0 "#PWR?" H 1850 2700 50  0001 C CNN
+F 0 "#PWR06" H 1850 2700 50  0001 C CNN
 F 1 "+3.3V" H 1865 3023 50  0000 C CNN
 F 2 "" H 1850 2850 50  0001 C CNN
@@
 	1850 3300 2550 3300
 $Comp
-L Device:C_Small C?
+L Device:C_Small C1
 U 1 1 5D8CAEE3
 P 1150 5150
-F 0 "C?" H 1250 5200 50  0000 L CNN
+F 0 "C1" H 1250 5200 50  0000 L CNN
 F 1 "1uF" H 1242 5105 50  0000 L CNN
 F 2 "" H 1150 5150 50  0001 C CNN
@@
 	850  5000 850  4950
 $Comp
-L power:GND #PWR?
+L power:GND #PWR05
 U 1 1 5D8CC801
 P 1150 5250
-F 0 "#PWR?" H 1150 5000 50  0001 C CNN
+F 0 "#PWR05" H 1150 5000 50  0001 C CNN
 F 1 "GND" H 1155 5077 50  0000 C CNN
 F 2 "" H 1150 5250 50  0001 C CNN
@@
 $EndComp
 $Comp
-L Device:R_Small_US R?
+L Device:R_Small_US R4
 U 1 1 5D8CCF3A
 P 2300 2500
-F 0 "R?" V 2095 2500 50  0000 C CNN
+F 0 "R4" V 2095 2500 50  0000 C CNN
 F 1 "100k" V 2186 2500 50  0000 C CNN
 F 2 "" H 2300 2500 50  0001 C CNN
@@
 	2100 2500 2100 2600
 $Comp
-L power:GND #PWR?
+L power:GND #PWR010
 U 1 1 5D8CEF8F
 P 2100 2600
-F 0 "#PWR?" H 2100 2350 50  0001 C CNN
+F 0 "#PWR010" H 2100 2350 50  0001 C CNN
 F 1 "GND" H 2105 2427 50  0000 C CNN
 F 2 "" H 2100 2600 50  0001 C CNN
@@
 	3450 3200 3150 3200
 Wire Wire Line
-	3450 3200 3850 3200
+	3450 3200 3600 3200
 Connection ~ 3450 3200
 $Comp
-L Device:R_POT_TRIM_US RV?
+L Device:R_POT_TRIM_US RV2
 U 1 1 5D8D08F7
 P 3000 2300
-F 0 "RV?" V 3050 2450 50  0000 C CNN
+F 0 "RV2" V 3050 2450 50  0000 C CNN
 F 1 "1M" V 2900 2300 50  0000 C CNN
 F 2 "" H 3000 2300 50  0001 C CNN
@@
 Loud
 $Comp
-L Device:R_POT_TRIM_US RV?
+L Device:R_POT_TRIM_US RV1
 U 1 1 5D8D3430
 P 2050 5050
-F 0 "RV?" V 2100 5200 50  0000 C CNN
+F 0 "RV1" V 2100 5200 50  0000 C CNN
 F 1 "1M" V 1950 5050 50  0000 C CNN
 F 2 "" H 2050 5050 50  0001 C CNN
@@
 $EndComp
 $Comp
-L power:+3.3V #PWR?
+L power:+3.3V #PWR08
 U 1 1 5D8D36A6
 P 2050 4750
-F 0 "#PWR?" H 2050 4600 50  0001 C CNN
+F 0 "#PWR08" H 2050 4600 50  0001 C CNN
 F 1 "+3.3V" H 2065 4923 50  0000 C CNN
 F 2 "" H 2050 4750 50  0001 C CNN
@@
 	2050 5200 2050 5350
 $Comp
-L power:GND #PWR?
+L power:GND #PWR09
 U 1 1 5D8D49B3
 P 2050 5350
-F 0 "#PWR?" H 2050 5100 50  0001 C CNN
+F 0 "#PWR09" H 2050 5100 50  0001 C CNN
 F 1 "GND" H 2055 5177 50  0000 C CNN
 F 2 "" H 2050 5350 50  0001 C CNN
@@
 	2300 4850 2650 4850
 Wire Wire Line
-	3250 4950 3700 4950
+	3250 4950 3600 4950
 Text Notes 2200 5350 0    50   ~ 0
 Comparator is to wake up the microcontroller.\nThis will help with power savings
 Text Notes 3050 6600 0    50   ~ 0
 Spares
+Wire Wire Line
+	3600 4950 3600 3700
+Wire Wire Line
+	3600 3700 6450 3700
+Connection ~ 3600 4950
+Wire Wire Line
+	3600 4950 3700 4950
+Wire Wire Line
+	3600 3200 3600 3600
+Wire Wire Line
+	3600 3600 6450 3600
+Connection ~ 3600 3200
+Wire Wire Line
+	3600 3200 3850 3200
+Text Notes 6750 4450 0    197  ~ 39
+STM32
 $EndSCHEMATC

Commit message: Added some parts to the schematic, maps some parts to their footprints. You know.
Parts:
- added C23, C24, C25: 1uF, Capacitor_SMD:C_0805_2012Metric, symbol Device:C_Small
- added J4: Conn_01x02_Male, Connector_PinHeader_2.54mm:PinHeader_1x02_P2.54mm_Vertical, symbol Connector:Conn_01x02_Male
- added R13, R14: 1M, Resistor_SMD:R_0805_2012Metric, symbol Device:R_Small_US
- added SW2, SW3: SW_Push_Dual, symbol Switch:SW_Push_Dual
- added U4: Si7050-A20, Package_DFN_QFN:DFN-6-1EP_3x3mm_P1mm_EP1.65x2.55mm, symbol Sensor_Temperature:Si7050-A20
- added U5: LTR-303ALS-01, OptoDevice:Lite-On_LTR-303ALS-01, symbol Sensor_Optical:LTR-303ALS-01
- BT1: footprint (none) -> Battery:BatteryHolder_Keystone_1042_1x18650
- C1, C2, C3, C4: footprint (none) -> Capacitor_SMD:C_0805_2012Metric
- R1, R2, R3, R4: footprint (none) -> Resistor_SMD:R_0805_2012Metric
- RV1, RV2: footprint (none) -> Potentiometer_SMD:Potentiometer_Bourns_3269W_Vertical; Part Number (none) -> 3269W-1-105GLF
- U1: footprint (none) -> Package_SO:SOIC-14_3.9x8.7mm_P1.27mm; Part Number (none) -> LM324DR
- U1: footprint (none) -> Package_SO:SOIC-14_3.9x8.7mm_P1.27mm
- U2: footprint (none) -> Package_TO_SOT_SMD:SOT-223-3_TabPin2
Connections:
- net +3V3: now also C24.1, C25.1, R13.1, R14.1, U4.5 (VDD), U5.1 (VDD)
- net Audio: no longer U1.5 (+)
- net GND: now also C23.1, C23.2, C24.2, C25.2, SW2.2, SW2.4, SW3.2, SW3.4, U4.2 (GND), U5.3 (GND)
- net at C3.1, U2.3 (VI): now also J4.1 (Pin_1); no longer BT1.1 (+)
- net Raw_Audio: now reaches C2.1, R2.2, R3.1, U1.3 (+)
- net Raw_Audio: now also U1.5 (+)
- new net: BT1.1 (+), J4.2 (Pin_2)
- new net PB1: SW2.1, SW2.3
- new net PB2: SW3.1, SW3.3
- new net SCL: R14.2, U4.1 (SDA), U5.4 (SCL)
- new net SDA: R13.2, U4.6 (SCL), U5.6 (SDA)
Other:
- note added: "Light Sensor"
- note added: "On Switch"
- note added: "Temp Sensor"
- moved on the sheet: C1, U1E

Commit message: Hardware is almost finished
Parts:
- removed C23: 1uF, Capacitor_SMD:C_0805_2012Metric, symbol Device:C_Small
- removed SW2, SW3: SW_Push_Dual, symbol Switch:SW_Push_Dual
- added J6: Conn_01x03_Male, Connector_PinHeader_2.54mm:PinHeader_1x03_P2.54mm_Vertical, symbol Connector:Conn_01x03_Male
- added SW2, SW3: KSA0A311 LFTR, Button_Switch_THT:SW_Tactile_Straight_KSA0Axx1LFTR, symbol Switch:SW_Push
- BT1: Part Number (none) -> 1042P
- MK1: footprint (none) -> Connector_PinHeader_2.54mm:PinHeader_1x02_P2.54mm_Vertical
- RV1, RV2: footprint Potentiometer_SMD:Potentiometer_Bourns_3269W_Vertical -> Potentiometer_THT:Potentiometer_Vishay_T73YP_Vertical; Part Number 3269W-1-105GLF -> 3362P-1-105LF
- U4: footprint Package_DFN_QFN:DFN-6-1EP_3x3mm_P1mm_EP1.65x2.55mm -> Package_DFN_QFN:DFN-6-1EP_3x3mm_P1mm_EP1.5x2.4mm
Connections:
- net GND: now also U1.10 (+), U1.9 (-), SW2.2, SW3.2
- net PB1: now also SW2.1
- net PB2: now also SW3.1
- net at R4.1, U1.2 (-): now also RV2.1; no longer RV2.3
- net at U1.12 (+): now also J6.3 (Pin_3)
- net at U1.13 (-): now also J6.2 (Pin_2)
- net at U1.14: now also J6.1 (Pin_1)
Other:
- moved on the sheet: U1D
Changed lines of the file:
@@
 EESchema Schematic File Version 4
 LIBS:birdEar-cache
-EELAYER 30 0
+EELAYER 26 0
 EELAYER END
 $Descr USLetter 11000 8500
@@
 F 0 "MK1" H 980 3746 50  0000 L CNN
 F 1 "CMA-4544PF-W" H 980 3655 50  0000 L CNN
-F 2 "" V 850 3800 50  0001 C CNN
+F 2 "Connector_PinHeader_2.54mm:PinHeader_1x02_P2.54mm_Vertical" V 850 3800 50  0001 C CNN
 F 3 "~" V 850 3800 50  0001 C CNN
 	1    850  3700
@@
 F 2 "Battery:BatteryHolder_Keystone_1042_1x18650" V 1200 1660 50  0001 C CNN
 F 3 "~" V 1200 1660 50  0001 C CNN
+F 4 "1042P" H 1200 1600 50  0001 C CNN "Part Number"
 	1    1200 1600
 	1    0    0    -1
@@
 L Amplifier_Operational:LM324 U1
 U 4 1 5D8C5409
-P 2900 7050
-F 0 "U1" H 2900 7417 50  0000 C CNN
-F 1 "LM324" H 2900 7326 50  0000 C CNN
-F 2 "Package_SO:SOIC-14_3.9x8.7mm_P1.27mm" H 2850 7150 50  0001 C CNN
-F 3 "http://www.ti.com/lit/ds/symlink/lm2902-n.pdf" H 2950 7250 50  0001 C CNN
-F 4 "LM324DR" H 2900 7050 50  0001 C CNN "Part Number"
-	4    2900 7050
+P 2900 7200
+F 0 "U1" H 2900 7567 50  0000 C CNN
+F 1 "LM324" H 2900 7476 50  0000 C CNN
+F 2 "Package_SO:SOIC-14_3.9x8.7mm_P1.27mm" H 2850 7300 50  0001 C CNN
+F 3 "http://www.ti.com/lit/ds/symlink/lm2902-n.pdf" H 2950 7400 50  0001 C CNN
+F 4 "LM324DR" H 2900 7200 50  0001 C CNN "Part Number"
+	4    2900 7200
 	1    0    0    -1
 $EndComp
@@
 	1    0    0    -1
 $EndComp
-Wire Wire Line
-	800  7450 800  7500
 $Comp
 L power:GND #PWR03
@@
 U 1 1 5D8D08F7
 P 3000 2300
-F 0 "RV2" V 3050 2450 50  0000 C CNN
+F 0 "RV2" V 2900 2150 50  0000 C CNN
 F 1 "1M" V 2900 2300 50  0000 C CNN
-F 2 "Potentiometer_SMD:Potentiometer_Bourns_3269W_Vertical" H 3000 2300 50  0001 C CNN
+F 2 "Potentiometer_THT:Potentiometer_Vishay_T73YP_Vertical" H 3000 2300 50  0001 C CNN
 F 3 "~" H 3000 2300 50  0001 C CNN
-F 4 "3269W-1-105GLF" V 3000 2300 50  0001 C CNN "Part Number"
+F 4 "3362P-1-105LF" V 3000 2300 50  0001 C CNN "Part Number"
 	1    3000 2300
-	0    1    1    0
+	0    -1   1    0
 $EndComp
 Wire Wire Line
@@
 F 0 "RV1" V 2100 5200 50  0000 C CNN
 F 1 "1M" V 1950 5050 50  0000 C CNN
-F 2 "Potentiometer_SMD:Potentiometer_Bourns_3269W_Vertical" H 2050 5050 50  0001 C CNN
+F 2 "Potentiometer_THT:Potentiometer_Vishay_T73YP_Vertical" H 2050 5050 50  0001 C CNN
 F 3 "~" H 2050 5050 50  0001 C CNN
-F 4 "3269W-1-105GLF" V 2050 5050 50  0001 C CNN "Part Number"
+F 4 "3362P-1-105LF" V 2050 5050 50  0001 C CNN "Part Number"
 	1    2050 5050
 	1    0    0    1
@@
 Text Notes 6750 4450 0    197  ~ 39
 STM32
-$Comp
-L Device:C_Small C23
-U 1 1 5D985D1A
-P 1100 7650
-F 0 "C23" H 1200 7700 50  0000 L CNN
-F 1 "1uF" H 1192 7605 50  0000 L CNN
-F 2 "Capacitor_SMD:C_0805_2012Metric" H 1100 7650 50  0001 C CNN
-F 3 "~" H 1100 7650 50  0001 C CNN
-	1    1100 7650
-	1    0    0    -1
-$EndComp
-Wire Wire Line
-	1100 7550 1100 7500
-Wire Wire Line
-	1100 7500 800  7500
-$Comp
-L power:GND #PWR032
-U 1 1 5D985D22
-P 1100 7750
-F 0 "#PWR032" H 1100 7500 50  0001 C CNN
-F 1 "GND" H 1105 7577 50  0000 C CNN
-F 2 "" H 1100 7750 50  0001 C CNN
-F 3 "" H 1100 7750 50  0001 C CNN
-	1    1100 7750
-	1    0    0    -1
-$EndComp
-Connection ~ 800  7500
-Wire Wire Line
-	800  7500 800  7600
 Text Label 2000 3300 0    50   ~ 0
 Raw_Audio
@@
 F 0 "U4" H 9144 3746 50  0000 L CNN
 F 1 "Si7050-A20" H 9144 3655 50  0000 L CNN
-F 2 "Package_DFN_QFN:DFN-6-1EP_3x3mm_P1mm_EP1.65x2.55mm" H 8800 3300 50  0001 C CNN
+F 2 "Package_DFN_QFN:DFN-6-1EP_3x3mm_P1mm_EP1.5x2.4mm" H 8800 3300 50  0001 C CNN
 F 3 "https://www.silabs.com/documents/public/data-sheets/Si7050-1-3-4-5-A20.pdf" H 8600 4000 50  0001 C CNN
 	1    8800 3700
@@
 Wire Wire Line
 	8800 4050 8800 4000
-$Comp
-L Switch:SW_Push_Dual SW?
-U 1 1 5D9F0852
-P 5400 5250
-AR Path="/5D8C399D/5D9F0852" Ref="SW?"  Part="1"
-AR Path="/5D9F0852" Ref="SW2"  Part="1"
-F 0 "SW2" H 5400 5535 50  0000 C CNN
-F 1 "SW_Push_Dual" H 5400 5444 50  0000 C CNN
-F 2 "" H 5400 5450 50  0001 C CNN
-F 3 "~" H 5400 5450 50  0001 C CNN
-	1    5400 5250
-	1    0    0    -1
-$EndComp
-Wire Wire Line
-	5200 5250 5100 5250
-Wire Wire Line
-	5100 5250 5100 5350
-Wire Wire Line
-	5100 5450 5200 5450
-Wire Wire Line
-	5600 5250 5700 5250
-Wire Wire Line
-	5700 5250 5700 5350
-Wire Wire Line
-	5700 5450 5600 5450
-Wire Wire Line
-	5700 5350 5900 5350
 Wire Wire Line
 	5900 5350 5900 5650
-Connection ~ 5700 5350
-Wire Wire Line
-	5700 5350 5700 5450
 $Comp
 L power:GND #PWR?
@@
 	1    0    0    -1
 $EndComp
-Wire Wire Line
-	5100 5350 4900 5350
-Connection ~ 5100 5350
-Wire Wire Line
-	5100 5350 5100 5450
 Text Label 4900 5350 0    50   ~ 0
 PB1
-$Comp
-L Switch:SW_Push_Dual SW?
-U 1 1 5D9F086C
-P 6600 5250
-AR Path="/5D8C399D/5D9F086C" Ref="SW?"  Part="1"
-AR Path="/5D9F086C" Ref="SW3"  Part="1"
-F 0 "SW3" H 6600 5535 50  0000 C CNN
-F 1 "SW_Push_Dual" H 6600 5444 50  0000 C CNN
-F 2 "" H 6600 5450 50  0001 C CNN
-F 3 "~" H 6600 5450 50  0001 C CNN
-	1    6600 5250
-	1    0    0    -1
-$EndComp
-Wire Wire Line
-	6400 5250 6300 5250
-Wire Wire Line
-	6300 5250 6300 5350
-Wire Wire Line
-	6300 5450 6400 5450
-Wire Wire Line
-	6800 5250 6900 5250
-Wire Wire Line
-	6900 5250 6900 5350
-Wire Wire Line
-	6900 5450 6800 5450
-Wire Wire Line
-	6900 5350 7100 5350
 Wire Wire Line
 	7100 5350 7100 5650
-Connection ~ 6900 5350
-Wire Wire Line
-	6900 5350 6900 5450
 $Comp
 L power:GND #PWR?
@@
 	1    0    0    -1
 $EndComp
-Wire Wire Line
-	6300 5350 6100 5350
-Connection ~ 6300 5350
-Wire Wire Line
-	6300 5350 6300 5450
 Text Label 6100 5350 0    50   ~ 0
 PB2
@@
 Text Notes 1450 750  0    50   ~ 0
 On Switch
+$Comp
+L Switch:SW_Push SW2
+U 1 1 5D9A7F57
+P 5400 5350
+F 0 "SW2" H 5400 5635 50  0000 C CNN
+F 1 "KSA0A311 LFTR" H 5400 5544 50  0000 C CNN
+F 2 "Button_Switch_THT:SW_Tactile_Straight_KSA0Axx1LFTR" H 5400 5550 50  0001 C CNN
+F 3 "" H 5400 5550 50  0001 C CNN
+	1    5400 5350
+	1    0    0    -1
+$EndComp
+$Comp
+L Switch:SW_Push SW3
+U 1 1 5D9A8159
+P 6600 5350
+F 0 "SW3" H 6600 5635 50  0000 C CNN
+F 1 "KSA0A311 LFTR" H 6600 5544 50  0000 C CNN
+F 2 "Button_Switch_THT:SW_Tactile_Straight_KSA0Axx1LFTR" H 6600 5550 50  0001 C CNN
+F 3 "" H 6600 5550 50  0001 C CNN
+	1    6600 5350
+	1    0    0    -1
+$EndComp
+Wire Wire Line
+	5600 5350 5900 5350
+Wire Wire Line
+	4900 5350 5200 5350
+Wire Wire Line
+	6100 5350 6400 5350
+Wire Wire Line
+	6800 5350 7100 5350
+Wire Wire Line
+	800  7450 800  7600
+$Comp
+L Connector:Conn_01x03_Male J6
+U 1 1 5DBAAF06
+P 2900 7750
+F 0 "J6" V 3053 7890 50  0000 L CNN
+F 1 "Conn_01x03_Male" V 2962 7890 50  0000 L CNN
+F 2 "Connector_PinHeader_2.54mm:PinHeader_1x03_P2.54mm_Vertical" H 2900 7750 50  0001 C CNN
+F 3 "~" H 2900 7750 50  0001 C CNN
+	1    2900 7750
+	0    1    -1   0
+$EndComp
+Wire Wire Line
+	3000 7550 3000 7450
+Wire Wire Line
+	3000 7450 3300 7450
+Wire Wire Line
+	3300 7450 3300 7200
+Wire Wire Line
+	3300 7200 3200 7200
+Wire Wire Line
+	2800 7550 2500 7550
+Wire Wire Line
+	2500 7550 2500 7100
+Wire Wire Line
+	2500 7100 2600 7100
+Wire Wire Line
+	2600 7300 2600 7450
+Wire Wire Line
+	2600 7450 2900 7450
+Wire Wire Line
+	2900 7450 2900 7550
+Wire Wire Line
+	2650 6150 2500 6150
+Wire Wire Line
+	2500 6150 2500 6350
+Wire Wire Line
+	2650 6350 2500 6350
+Connection ~ 2500 6350
+Wire Wire Line
+	2500 6350 2500 6650
+$Comp
+L power:GND #PWR0105
+U 1 1 5DBC4ABE
+P 2500 6650
+F 0 "#PWR0105" H 2500 6400 50  0001 C CNN
+F 1 "GND" H 2505 6477 50  0000 C CNN
+F 2 "" H 2500 6650 50  0001 C CNN
+F 3 "" H 2500 6650 50  0001 C CNN
+	1    2500 6650
+	1    0    0    -1
+$EndComp
 $EndSCHEMATC
